File: npm1300.kicad_sch (KiCad schematic)
At the start: 29 parts, among them J5 JST_PH_S2B-PH-SM4, SW2 B3U-1000P, U10 nPM1300-QEXX, U11 TPS22917DBV, U12 TPS63031DSK, U9 TLV73311PDBV

Commit message: mostly finished; just need to breakout extra gpio
Parts:
- removed C38, C39: 1uF, Capacitor_SMD:C_0402_1005Metric, symbol Device:C_Small
- removed C45: 10uF, Capacitor_SMD:C_0402_1005Metric, symbol Device:C_Small
- removed C50: 1nF, Capacitor_SMD:C_0402_1005Metric, symbol Device:C_Small
- removed L1: 2.2uH, Inductor_SMD:L_0603_1608Metric, symbol Device:L_Small
- removed R16: 47k, Resistor_SMD:R_0402_1005Metric, symbol Device:R_Small
- removed U11: TPS22917DBV, Package_TO_SOT_SMD:SOT-23-6, symbol Power_Management:TPS22917DBV
- removed U9: TLV73311PDBV, Package_TO_SOT_SMD:SOT-23-5, symbol Regulator_Linear:TLV73311PDBV
- added C35: 1nF, Capacitor_SMD:C_0603_1608Metric, symbol Device:C_Small
- added U6: TPS22917DBV, Package_TO_SOT_SMD:SOT-23-6, symbol Power_Management:TPS22917DBV
- C25: renamed from C37; footprint Capacitor_SMD:C_0402_1005Metric -> Capacitor_SMD:C_0603_1608Metric
- C26: renamed from C40; footprint Capacitor_SMD:C_0402_1005Metric -> Capacitor_SMD:C_0603_1608Metric
- C31: renamed from C46; footprint Capacitor_SMD:C_0402_1005Metric -> Capacitor_SMD:C_0603_1608Metric
- C32: renamed from C47; footprint Capacitor_SMD:C_0402_1005Metric -> Capacitor_SMD:C_0603_1608Metric
- C33: renamed from C48; footprint Capacitor_SMD:C_0402_1005Metric -> Capacitor_SMD:C_0603_1608Metric
- C34: renamed from C49; footprint Capacitor_SMD:C_0402_1005Metric -> Capacitor_SMD:C_0603_1608Metric
- C36: renamed from C51; footprint Capacitor_SMD:C_0402_1005Metric -> Capacitor_SMD:C_0603_1608Metric
- C37: renamed from C52; footprint Capacitor_SMD:C_0402_1005Metric -> Capacitor_SMD:C_0603_1608Metric
- C38: renamed from C53; footprint Capacitor_SMD:C_0402_1005Metric -> Capacitor_SMD:C_0603_1608Metric
- C39: renamed from C54; footprint Capacitor_SMD:C_0402_1005Metric -> Capacitor_SMD:C_0603_1608Metric
- J4: renamed from J5; symbol Connector_Generic:Conn_01x02 -> Connector_Generic_MountingPin:Conn_01x02_MountingPin
- SW3: renamed from SW2; footprint Button_Switch_SMD:SW_SPST_B3U-1000P -> Button_Switch_SMD:SW_Push_1P1T_NO_Vertical_Wuerth_434133025816
- renumbered C41 to C27, C42 to C28, C43 to C29, C44 to C30, U10 to U5, U12 to U7
Connections:
- net +3V3: now also C26.1, D1.2 (A), D2.2 (A), U5.12 (VDDIO), C35.1, U6.1 (VIN)
- net GND: now also J4.MP (MountPin), U5.17 (VSET1), U6.2 (GND)
- net SD_ON: now also U6.3 (ON)
- net SD_VCC: now also U6.5 (QOD), U6.6 (VOUT)
- net VSYS: now also U5.1 (VOUT1)
- removed net +1V8: C26.1, D1.2 (A), D2.2 (A), U5.1 (VOUT1), U5.12 (VDDIO)
- new net: C35.2, U6.4 (CT)
- no-connect marks 2 -> 3
Other:
- note added: "Buck 1 off at startup"
- note added: "Buck 2 off at startup"
- note removed: "1.8v -> 1.1v Linear Regulator"
- note removed: "Buck 1 1.8v at startup"
- note removed: "Buck 2 off on startup"
- moved on the sheet: SW3
