File: npm1300.kicad_sch (KiCad schematic)
At the start: 23 parts, among them J4 JST_PH_S2B-PH-SM4, SW3 B3U-1000P, U5 nPM1300-QEXX, U6 TPS22917DBV, U7 TPS63031DSK

Commit message: v2.1
Parts:
- removed C27, C29, C31: 10uF, Capacitor_SMD:C_0603_1608Metric, symbol Device:C_Small
- removed C28, C30, C33: 100nF, Capacitor_SMD:C_0603_1608Metric, symbol Device:C_Small
- removed C32: 2.2uF, Capacitor_SMD:C_0603_1608Metric, symbol Device:C_Small
- removed C34: 1uF, Capacitor_SMD:C_0603_1608Metric, symbol Device:C_Small
- removed SW3: B3U-1000P, Button_Switch_SMD:SW_Push_1P1T_NO_Vertical_Wuerth_434133025816, symbol Switch:SW_Push
- removed U5: nPM1300-QEXX, Package_DFN_QFN:QFN-32-1EP_5x5mm_P0.5mm_EP3.6x3.6mm_ThermalVias, symbol PCM_nordic-lib-kicad-npm:nPM1300-QEXX
- added C19: 100nF, Capacitor_SMD:C_0603_1608Metric, symbol Device:C_Small
- added C40: 1nF, Capacitor_SMD:C_0603_1608Metric, symbol Device:C_Small
- added C41, C42: 1uF, Capacitor_SMD:C_0603_1608Metric, symbol Device:C_Small
- added D3: B5819W SL, Diode_SMD:D_SOD-123, symbol Device:D_Small
- added Q1: AO3401A, Package_TO_SOT_SMD:SOT-23, symbol Transistor_FET:AO3401A
- added R16, R17: 100k, Resistor_SMD:R_0603_1608Metric, symbol Device:R_Small
- added R18: 3k, Resistor_SMD:R_0603_1608Metric, symbol Device:R_Small
- added R19, R20: 1k, Resistor_SMD:R_0603_1608Metric, symbol Device:R_Small
- added R21: 1M, Resistor_SMD:R_0603_1608Metric, symbol Device:R_Small
- added R22: 470k, Resistor_SMD:R_0603_1608Metric, symbol Device:R_Small
- added R23: 10k, Resistor_SMD:R_0603_1608Metric, symbol Device:R_Small
- added U5: TP4056-42-ESOP8, Package_SO:SOIC-8-1EP_3.9x4.9mm_P1.27mm_EP2.41x3.3mm_ThermalVias, symbol Battery_Management:TP4056-42-ESOP8
- added U8: TPS22917DBVR, Package_TO_SOT_SMD:SOT-23-6, symbol Power_Management:TPS22917DBV
- C25: value 1uF -> 4.7uF; LCSC PN (none) -> C19666
- C26: value 100nF -> 10uF; LCSC PN (none) -> C96446
- C36: value 10uF -> 4.7uF; LCSC PN (none) -> C19666
- D1: value LED0 -> Yellow; footprint LED_SMD:LED_1206_3216Metric_Pad1.42x1.75mm_HandSolder -> LED_SMD:LED_0805_2012Metric; LCSC PN (none) -> C2296
- D2: value LED1 -> Green; footprint LED_SMD:LED_1206_3216Metric_Pad1.42x1.75mm_HandSolder -> LED_SMD:LED_0805_2012Metric; LCSC PN (none) -> C2297
- J4: value JST_PH_S2B-PH-SM4 -> S2B-PH-SM4-TB(LF)(SN)
- L1: renamed from L2; value 2.2uH -> 1.5uH; footprint Inductor_SMD:L_0603_1608Metric -> Inductor_SMD:L_Murata_DFE201610P; LCSN PN C6079477 -> (none); Part Number LSCNB1608HKT2R2MD -> DFE201610E-1R5M=P2
- U6: value TPS22917DBV -> TPS22917DBVR; LCSC PN C2680344 -> (none)
- U7: value TPS63031DSK -> TPS63031DSKR; Part Number (none) -> TPS63031DSKR
Connections:
- net +3V3: now also C40.1, C41.1, C42.1, U8.1 (VIN); no longer C26.1, D1.2 (A), D2.2 (A)
- net +BATT: now also C26.1, Q1.3 (D), R21.1, U5.5 (BAT)
- net GND: now also C19.2, C41.2, C42.2, R16.2, R17.2, R18.2, R22.2, R23.2, U5.1 (TEMP), U5.3 (GND), U5.9 (EPAD), U8.2 (GND)
- net SD_ON: now also R16.1
- net VBUS: now also D3.2 (A), Q1.1 (G), R19.1, R20.1, R23.1, U5.4 (V_{CC}), U5.8 (CE)
- net VSYS: now also D3.1 (K), Q1.2 (S)
- net at D2.1 (K): now also U5.6 (~{STDBY})
- net at D1.1 (K): now also U5.7 (~{CHRG})
- new net: D2.2 (A), R20.2
- new net: R18.1, U5.2 (PROG)
- new net: C40.2, U8.4 (CT)
- new net: D1.2 (A), R19.2
- new net BATT_SENSE: C19.1, R21.2, R22.1
- new net DISP_ON: R17.1, U8.3 (ON)
- new net DISP_VCC: U8.5 (QOD), U8.6 (VOUT)
- no-connect marks 3 -> 0
Other:
- note added: "Disp Load Switch"
- note added: "Power Circuits 3.3v from TPS63031"
- note removed: "Buck 1 off at startup"
- note removed: "Buck 2 off at startup"
- note removed: "Power Circuits 3.3v from TPS63031 1.8v from npm1300 1.1v via linear regulator"
- note removed: "Ship/Hibernate Button"
- moved on the sheet: C25, C35, C36, C37, D1, D2, U6
