File: dap-proto-board-full.kicad_pcb (KiCad board)
At the start: 4 copper layers, 45.8 x 61.4 mm, 73 parts, among them J1 SFV18R-1STE1HLF, J2 UJ20-C-H-G-SMT-1-P16-TR, J3 SJ-3523-SMT, J4 JST_PH_S2B-PH-SM4, J5 Conn_01x14, SW1 SW_Push, SW2 SW_Push, SW3 B3U-1000P, U1 MSD-11-A, U2 USBLC6-2SC6, U3 TAD5212, U4 ESP32-S3, U5 nPM1300-QEXX, U6 TPS22917DBV, U7 TPS63031DSK, Y1 ABM8-40.000MHZ-12-B1U-T

Commit message: v2.1
Parts:
- removed C27, C29, C31: 10uF, Capacitor_SMD:C_0603_1608Metric
- removed C28, C30, C33: 100nF, Capacitor_SMD:C_0603_1608Metric
- removed C32: 2.2uF, Capacitor_SMD:C_0603_1608Metric
- removed C34: 1uF, Capacitor_SMD:C_0603_1608Metric
- removed SW3: B3U-1000P, Button_Switch_SMD:SW_Push_1P1T_NO_Vertical_Wuerth_434133025816
- added C19: 100nF, Capacitor_SMD:C_0603_1608Metric, F.Cu at (123.4, 77.2)
- added C40: 1nF, Capacitor_SMD:C_0603_1608Metric, F.Cu at (97.3, 74.5)
- added C41: 1uF, Capacitor_SMD:C_0603_1608Metric, F.Cu at (104.0, 78.4)
- added C42: 1uF, Capacitor_SMD:C_0603_1608Metric, F.Cu at (114.2, 95.2)
- added D3: B5819W SL, Diode_SMD:D_SOD-123, F.Cu at (116.7, 75.5)
- added Q1: AO3401A, Package_TO_SOT_SMD:SOT-23, F.Cu at (120.0, 75.8)
- added R14: 22, Resistor_SMD:R_0603_1608Metric, F.Cu at (111.8, 73.4)
- added R15: 10k, Resistor_SMD:R_0603_1608Metric, F.Cu at (128.6, 86.2)
- added R16: 100k, Resistor_SMD:R_0603_1608Metric, F.Cu at (111.0, 94.7)
- added R17: 100k, Resistor_SMD:R_0603_1608Metric, F.Cu at (101.5, 72.3)
- added R18: 3k, Resistor_SMD:R_0603_1608Metric, F.Cu at (121.5, 64.7)
- added R19: 1k, Resistor_SMD:R_0603_1608Metric, F.Cu at (120.5, 60.0)
- added R20: 1k, Resistor_SMD:R_0603_1608Metric, F.Cu at (124.0, 60.0)
- added R21: 1M, Resistor_SMD:R_0603_1608Metric, F.Cu at (125.6, 74.3)
- added R22: 470k, Resistor_SMD:R_0603_1608Metric, F.Cu at (125.6, 77.8)
- added R23: 10k, Resistor_SMD:R_0603_1608Metric, F.Cu at (116.8, 71.1)
- added R3: 22, Resistor_SMD:R_0603_1608Metric, F.Cu at (113.5, 73.4)
- added U8: TPS22917DBVR, Package_TO_SOT_SMD:SOT-23-6, F.Cu at (101.1, 75.9)
- C17, C18: value 18pF -> 15pF
- C25: value 1uF -> 4.7uF
- C26: value 100nF -> 10uF
- C36: value 10uF -> 4.7uF
- D1: value LED0 -> Yellow; footprint LED_SMD:LED_1206_3216Metric_Pad1.42x1.75mm_HandSolder -> LED_SMD:LED_0805_2012Metric
- D2: value LED1 -> Green; footprint LED_SMD:LED_1206_3216Metric_Pad1.42x1.75mm_HandSolder -> LED_SMD:LED_0805_2012Metric
- J3: value SJ-3523-SMT -> SJ-3523-SMT-TR
- J4: value JST_PH_S2B-PH-SM4 -> S2B-PH-SM4-TB(LF)(SN)
- L1: renamed from L2; value 2.2uH -> 1.5uH; footprint Inductor_SMD:L_0603_1608Metric -> Inductor_SMD:L_Murata_DFE201610P
- R10, R11: value 47k -> 5.1k
- R12, R13: value 47k -> 10k
- R4: value 2.2 -> 0
- U4: value ESP32-S3 -> ESP32-S3FH4R2
- U5: value nPM1300-QEXX -> TP4056-42-ESOP8; footprint Package_DFN_QFN:QFN-32-1EP_5x5mm_P0.5mm_EP3.6x3.6mm_ThermalVias -> Package_SO:SOIC-8-1EP_3.9x4.9mm_P1.27mm_EP2.41x3.3mm_ThermalVias
- U6: value TPS22917DBV -> TPS22917DBVR
- U7: value TPS63031DSK -> TPS63031DSKR
- Y1: value ABM8-40.000MHZ-12-B1U-T -> TSX-3225 40.0000MF15Y-K3
- moved D2 23.7 mm to (125.8, 58.0)
- moved R10 21.2 mm to (107.8, 65.8)
- moved D1 18.1 mm to (120.8, 58.0)
- moved R11 12.4 mm to (115.5, 66.8), turned to -90 degrees
- moved C25 9.50 mm to (119.8, 73.0), turned to 0 degrees
- moved C26 4.23 mm to (122.8, 73.5), turned to 90 degrees
- moved U5 3.60 mm to (123.8, 68.5), turned to 0 degrees
- moved C22 1.00 mm to (105.5, 78.4)
- moved C21 0.55 mm to (107.0, 78.4)
- moved L1 0.52 mm to (103.7, 72.7)
- moved J3 0.45 mm to (130.2, 111.8)
Connections:
- net /GPIO43 renamed /UART_TX
- net /GPIO44 renamed /UART_RX
- C21 pad 1: +3V3 -> Net-(U4-VDD_SPI)
- C22 pad 1: +3V3 -> Net-(U4-VDD_SPI)
- C26 pad 1: +3V3 -> +BATT
- D1 pad 2: +3V3 -> Net-(D1-A)
- D2 pad 2: +3V3 -> Net-(D2-A)
- J1 pad 1: +3V3 -> DISP_VCC
- J2 pad A5: /CC1 -> Net-(J2-CC1)
- J2 pad B5: /CC2 -> Net-(J2-CC2)
- J5 pad 6: /GPIO16 -> GND
- J5 pad 7: /GPIO15 -> GND
- R10 pad 1: +3V3 -> Net-(J2-CC2)
- R10 pad 2: /npm_SCL -> GND
- R11 pad 1: +3V3 -> Net-(J2-CC1)
- R11 pad 2: /npm_SDA -> GND
- R5 pad 1: +3V3 -> SD_VCC
- R6 pad 1: +3V3 -> SD_VCC
- R7 pad 1: +3V3 -> SD_VCC
- R8 pad 1: +3V3 -> SD_VCC
- R9 pad 1: +3V3 -> SD_VCC
- U3 pad 12: /tad_GPI1 -> GND
- U4 pad 15: /npm_SCL -> /BATT_SENSE
- U4 pad 16: /npm_SDA -> /GPIO11
- U4 pad 17: /npm_GPIO1 -> /GPIO12
- U4 pad 21: /GPIO15 -> /disp_CS
- U4 pad 22: /GPIO16 -> /DISP_ON
- U4 pad 25: /USB_D- -> Net-(U4-GPIO19/USB_D-)
- U4 pad 26: /USB_D+ -> Net-(U4-GPIO20/USB_D+)
- U4 pad 29: +3V3 -> Net-(U4-VDD_SPI)
- U4 pad 42: /disp_CS -> /disp_RESET
- U5 pad 1: VSYS -> GND
- U5 pad 2: GND -> Net-(U5-PROG)
- U5 pad 3: unconnected-(U5-SW1-Pad3) -> GND
- U5 pad 4: VSYS -> VBUS
- U5 pad 5: unconnected-(U5-SW2-Pad5) -> +BATT
- U5 pad 6: GND -> Net-(D2-K)
- U5 pad 7: /npm_GPIO0 -> Net-(D1-K)
- U5 pad 8: /npm_GPIO1 -> VBUS
- U5 pad 9: /npm_GPIO2 -> GND
Routing:
- net /GPIO16: track 29.1 -> 0.00 mm, vias 1 -> 0
- net /GPIO15: track 28.8 -> 0.00 mm, vias 1 -> 0
- net /npm_SCL: track 23.5 -> 0.00 mm
- net /npm_SDA: track 21.1 -> 0.00 mm
- net GND: track 123.0 -> 103.3 mm
- net /npm_GPIO1: track 17.5 -> 0.00 mm
- net /DISP_ON: track 0.00 -> 14.7 mm, vias 0 -> 2
- net VCOM: track 17.1 -> 31.3 mm, vias 3 -> 4
- net /BATT_SENSE: track 0.00 -> 14.0 mm
- net VBUS: track 15.0 -> 28.4 mm
- net /disp_RESET: track 0.00 -> 11.6 mm
- net /CC2: track 10.6 -> 0.00 mm, vias 2 -> 0
- net /SHPHLD: track 10.3 -> 0.00 mm
- net +3V3: track 36.0 -> 26.6 mm, vias 32 -> 26
- net /CC1: track 8.11 -> 0.00 mm
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- added copper zone on F.Cu, net DISP_VCC
- added copper zone on F.Cu, net Net-(U7-L1)
- added copper zone on F.Cu, net Net-(U7-L2)
Other:
- board text added: "Full DAP Proto Board v2.1 2026 Isaiah Gamble"
- board text added: "RX"
- board text added: "TX"
- board text removed: "43"
- board text removed: "44"
- board text removed: "Full DAP Proto Board v2 2026 Isaiah Gamble"
