File: dap-proto-board-full.kicad_sch (KiCad schematic)
At the start: 48 parts, among them J1 SFV18R-1STE1HLF, J2 UJ20-C-H-G-SMT-1-P16-TR, J3 SJ-3523-SMT, J5 Conn_01x14, SW1 SW_Push, SW2 SW_Push, U1 MSD-11-A, U2 USBLC6-2SC6, U3 TAD5212, U4 ESP32-S3, Y1 ABM8-40.000MHZ-12-B1U-T

Commit message: v2.1
Parts:
- added R14, R3: 22, Resistor_SMD:R_0603_1608Metric, symbol Device:R_Small
- added R15: 10k, Resistor_SMD:R_0603_1608Metric, symbol Device:R_Small
- C17, C18: value 18pF -> 15pF
- J2: LCSC PN C2988369 -> (none)
- J3: value SJ-3523-SMT -> SJ-3523-SMT-TR
- R10, R11: value 47k -> 5.1k
- R12, R13: value 47k -> 10k
- R4: value 2.2 -> 0
- SW1, SW2: Part Number (none) -> PTS810SJM250SMTR LFS
- U1: LCSC PN C22467016 -> (none)
- U3: LCSC PN C45068920 -> (none)
- U4: value ESP32-S3 -> ESP32-S3FH4R2; Part Number (none) -> ESP32-S3FH4R2
- Y1: value ABM8-40.000MHZ-12-B1U-T -> TSX-3225 40.0000MF15Y-K3; LCSC PN C20625731 -> (none)
Connections:
- net tad_GPI1 is gone; now on net GND: U3.12 (GPI1)
- net +3V3: now also R15.1; no longer C21.1, C22.1, J1.1 (Pin_1), R10.1, R11.1, R5.1, R6.1, R7.1, R8.1, R9.1, U4.29 (VDD_SPI)
- net GND: now also J5.6 (Pin_6), J5.7 (Pin_7), R10.2, R11.2
- net SD_VCC: now also R5.1, R6.1, R7.1, R8.1, R9.1
- net USB_D+: now also R14.1; no longer U4.26 (GPIO20/USB_D+)
- net USB_D-: now also R3.1; no longer U4.25 (GPIO19/USB_D-)
- net disp_CS: now also U4.21 (XTAL_32K_P); no longer U4.42 (GPIO37)
- net disp_RESET: now also U4.42 (GPIO37)
- net at SW1.2, U4.5 (GPIO0): now also R15.2
- net CC1: no longer names the net of J2.A5 (CC1)
- net CC1: now also R11.1
- net CC2: no longer names the net of J2.B5 (CC2)
- net CC2: now also R10.1
- removed net GPIO15: J5.7 (Pin_7), U4.21 (XTAL_32K_P)
- net GPIO16 renamed DISP_ON
- net DISP_ON: no longer J5.6 (Pin_6)
- net GPIO43 renamed UART_TX
- net GPIO44 renamed UART_RX
- net npm_GPIO1 renamed GPIO12
- net npm_SCL renamed BATT_SENSE
- net BATT_SENSE: no longer R10.2
- net npm_SDA renamed GPIO11
- net GPIO11: no longer R11.2
- new net: R14.2, U4.26 (GPIO20/USB_D+)
- new net: R3.2, U4.25 (GPIO19/USB_D-)
- new net: C21.1, C22.1, U4.29 (VDD_SPI)
- new net DISP_VCC: J1.1 (Pin_1)
- no-connect marks 24 -> 25
Other:
- note removed: "Series cap to reach 15pF capacitance for oscillator"
- moved on the sheet: R7, R8, R9, SW1
